Commit message: sensor snippets modified

File: uuv_sensor_plugins/uuv_sensor_ros_plugins/urdf/magnetometer_snippets.xacro (robot description, xacro)
@@ -52,9 +52,4 @@
         <origin xyz="0 0 0" rpy="0 0 0" />
       </inertial>
-      <visual>
-        <geometry>
-          <box size="0.1 0.1 0.1" />
-        </geometry>
-      </visual>
       <xacro:no_collision/>
     </link>

File: uuv_sensor_plugins/uuv_sensor_ros_plugins/urdf/pressure_snippets.xacro (robot description, xacro)
@@ -34,5 +34,6 @@
       estimateDepth="false"
       standardPressure="101.325"
-      kPaPerM="9.80638">
+      kPaPerM="9.80638"
+      scale="1">
       <inertia ixx="0.00001" ixy="0.0" ixz="0.0" iyy="0.00001" iyz="0.0" izz="0.00001" />
       <xacro:insert_block name="origin" />>
@@ -52,5 +53,6 @@
       estimateDepth="false"
       standardPressure="101.325"
-      kPaPerM="9.80638">
+      kPaPerM="9.80638"
+      scale="1">
       <inertia ixx="0.00001" ixy="0.0" ixz="0.0" iyy="0.00001" iyz="0.0" izz="0.00001" />
       <xacro:insert_block name="origin" />
@@ -58,5 +60,5 @@
   </xacro:macro>
   <xacro:macro name="pressure_plugin_macro"
-    params="namespace suffix parent_link topic mass update_rate
+    params="namespace suffix parent_link topic scale mass update_rate
       range noise_sigma noise_amplitude estimateDepth standardPressure kPaPerM
       *inertia *origin">
@@ -69,5 +71,5 @@
       <visual>
         <geometry>
-          <mesh filename="file://$(find uuv_sensor_ros_plugins)/meshes/pressure.dae" scale="1 1 1"/>
+          <mesh filename="file://$(find uuv_sensor_ros_plugins)/meshes/pressure.dae" scale="${scale} ${scale} ${scale}"/>
         </geometry>
       </visual>
